File: hardware/LamhKicad/Foinse.kicad_sch (KiCad schematic)
At the start: 120 parts, among them J1 Conn_ARM_JTAG_SWD_10, J2 2060-1452/998-404, J3 ESQ-110-14-G-D, J4 2060-1452/998-404, J5 2060-1452/998-404, J6 2060-1452/998-404, J7 2060-1452/998-404, J8 2601-1108, Q1 AO3400A, Q10 AO3400A, Q11 AO3400A, Q12 AO3400A, Q2 AO3400A, Q3 AO3400A, Q4 AO3400A, Q5 AO3400A, Q6 AO3400A, Q7 AO3400A, Q8 AO3400A, Q9 AO3400A, U1 STM32F072C8Tx, U10 LTV-817, U11 LTV-817, U12 LTV-817, U13 LTV-817, U2 TLV70433DBVT, U3 LTV-817, U4 TJA1051T-3, U5 TPS563203, U6 TPS563203, U7 LTV-817, U8 LTV-817, U9 LTV-817

Commit message: clean asf
Parts:
- removed C10: 100nF, symbol Device:C
- removed C11: 1 uF, symbol Device:C
- removed U2: TLV70433DBVT, TLV70433DBVT:DBV0005A_N, symbol TLV70433DBVT:TLV70433DBVT
