File: hardware/LamhKicad/KicadProject.kicad_pcb (KiCad board)
At the start: 6 copper layers, 60 x 60 mm, 83 parts, among them J1 5023860570, J2 436500303, J3 436500303, J4 436500303, J5 ESQ-110-X-X-D, J6 436500303, J7 EBBA-02-C-SS-BU, U1 TJA1051T-3, U2 PCA9685PW_112, U3 MPM3650CGQW-P, U4 STM32F072C8Tx, U5 TLV75533PDRV

Commit message: ready
Parts:
- added G***: LOGO, LOGO, F.Cu at (210.2, 120.8)
- C13, C17, C22, C23, C24, C26, C29, C3, C30, C6: footprint Capacitor_SMD:C_0402_1005Metric -> Capacitor_SMD:C_0603_1608Metric
- C16, C18, C19, C20: footprint Capacitor_THT:CP_Radial_D10.0mm_P5.00mm -> footprints:CAP_16SVPF1000MX
- moved C31 5.53 mm to (207.0, 112.6), turned to 90 degrees
- moved G*** 3.00 mm to (216.8, 121.2)
- moved C5 2.99 mm to (190.8, 114.1)
- moved C19 2.15 mm to (201.8, 84.4)
- moved C16 2.09 mm to (190.6, 84.1), turned to -135 degrees
- moved R6 2.00 mm to (189.5, 91.8), turned to 45 degrees
- moved C20 1.52 mm to (178.2, 95.7)
- moved C18 1.26 mm to (178.4, 83.9)
- moved C4 1.24 mm to (194.0, 104.1)
- moved C3 0.98 mm to (195.3, 104.0)
- moved C30 0.85 mm to (202.2, 115.0)
- moved C23 0.77 mm to (193.6, 114.0)
- moved C24 0.67 mm to (206.7, 115.1)
- moved C7 0.57 mm to (182.4, 101.1), turned to 180 degrees
- moved C13 0.45 mm to (182.0, 109.8)
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- renumbered 3V3 to 3v3
Routing:
- net Net-(C6-Pad1): track 0.00 -> 2.95 mm
- net Net-(U2-LED6): track 1.80 -> 3.95 mm
- net Net-(J3-Pad1): track 37.6 -> 35.5 mm
- net 5V_LOGIC: track 58.0 -> 59.3 mm
- net CAN_-: track 13.7 -> 12.8 mm
- net CAN_+: track 13.5 -> 12.8 mm
- net GND: track 27.8 -> 28.2 mm, vias 102 -> 104
