File: hardware/LamhKicad/KicadProject.kicad_sch (KiCad schematic)
At the start: 61 parts, among them J1 5023860570, J2 436500303, J3 436500303, J4 436500303, J5 ESQ-110-X-X-D, J6 436500303, J7 EBBA-02-C-SS-BU, U1 TJA1051T-3, U2 PCA9685PW_112, U4 STM32F072C8Tx

Commit message: ready for review the twost
Changed lines of the file:
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@@
 	(text "cable\n"
 		(exclude_from_sim no)
-		(at 69.342 218.948 0)
+		(at 215.9 181.864 0)
 		(effects
 			(font
@@
 	(text "https://www.digikey.com/en/products/detail/molex/0436500303/269000?s=N4IgTCBcDaICwGYBsBWADGhmQF0C+QA"
 		(exclude_from_sim no)
-		(at 123.952 231.14 0)
+		(at 270.51 194.056 0)
 		(effects
 			(font
@@
 	(text "https://www.digikey.ie/en/products/detail/molex/1451320303/9742477"
 		(exclude_from_sim no)
-		(at 102.616 222.25 0)
+		(at 249.174 185.166 0)
 		(effects
 			(font
@@
 	(text "connector\n"
 		(exclude_from_sim no)
-		(at 71.374 227.076 0)
+		(at 217.932 189.992 0)
 		(effects
 			(font

Commit message: ready
Parts:
- C13, C17, C3, C6: footprint Capacitor_SMD:C_0402_1005Metric -> Capacitor_SMD:C_0603_1608Metric
- C16, C18, C19, C20: footprint Capacitor_THT:CP_Radial_D10.0mm_P5.00mm -> CAP_16SVPF1000MX
Changed lines of the file:
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@@
 			)
 		)
-		(property "Footprint" "Capacitor_THT:CP_Radial_D10.0mm_P5.00mm"
+		(property "Footprint" "CAP_16SVPF1000MX"
 			(at 168.91 167.64 0)
 			(effects
@@
 			)
 		)
-		(property "Footprint" "Capacitor_SMD:C_0402_1005Metric"
+		(property "Footprint" "Capacitor_SMD:C_0603_1608Metric"
 			(at 171.1452 119.38 0)
 			(effects
@@
 			)
 		)
-		(property "Footprint" "Capacitor_THT:CP_Radial_D10.0mm_P5.00mm"
+		(property "Footprint" "CAP_16SVPF1000MX"
 			(at 173.99 167.64 0)
 			(effects
@@
 			)
 		)
-		(property "Footprint" "Capacitor_THT:CP_Radial_D10.0mm_P5.00mm"
+		(property "Footprint" "CAP_16SVPF1000MX"
 			(at 163.83 167.64 0)
 			(effects
@@
 			)
 		)
-		(property "Footprint" "Capacitor_THT:CP_Radial_D10.0mm_P5.00mm"
+		(property "Footprint" "CAP_16SVPF1000MX"
 			(at 179.07 167.64 0)
 			(effects
@@
 			)
 		)
-		(property "Footprint" "Capacitor_SMD:C_0402_1005Metric"
+		(property "Footprint" "Capacitor_SMD:C_0603_1608Metric"
 			(at 156.21 79.7052 0)
 			(effects
@@
 			)
 		)
-		(property "Footprint" "Capacitor_SMD:C_0402_1005Metric"
+		(property "Footprint" "Capacitor_SMD:C_0603_1608Metric"
 			(at 265.7348 63.5 0)
 			(effects
@@
 			)
 		)
-		(property "Footprint" "Capacitor_SMD:C_0402_1005Metric"
+		(property "Footprint" "Capacitor_SMD:C_0603_1608Metric"
 			(at 103.8352 60.96 0)
 			(effects
