File: hardware/LamhKicad/power.kicad_sch (KiCad schematic)
At the start: 22 parts, among them U3 MPM3650CGQW-P

Commit message: clean asf
Parts:
- removed C32: 4.7uf, Capacitor_SMD:C_0402_1005Metric, symbol Device:C
- removed R17, R18: 0Ω, Resistor_SMD:R_0402_1005Metric, symbol Device:R
- removed R19: 499kΩ, Resistor_SMD:R_0402_1005Metric, symbol Device:R
- removed R21: 33.2kΩ, Resistor_SMD:R_0402_1005Metric, symbol Device:R
- removed VR1: LT3045EDD_PBF, SON50P300X300X80-11N, symbol LT3045EDD_PBF:LT3045EDD_PBF
- added U5: TLV75533PDRV, Package_SON:WSON-6-1EP_2x2mm_P0.65mm_EP1x1.6mm, symbol Regulator_Linear:TLV75533PDRV
- C32: renamed from C33; value 4.7uf -> 1uf
- C33: renamed from C34; value 10uf -> 1uf
- renumbered C31 to C24, C30 to C26, C26 to C30, C24 to C31, R20 to R17
Connections:
- net AGND is gone; now on net GND: C25.1, R15.1, U3.18 (AGND)
- net 3.3v: now also U5.1 (OUT)
- net GND: now also U5.3 (GND), U5.7 (GND)
- net vin: now also U3.16 (EN)
- net at C2.2, R15.2, R16.1: now also U3.17 (FB)
- net at C2.1, C24.1, C26.1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: now also U5.4 (EN), U5.6 (IN)
- no-connect marks 8 -> 7
Other:
- note added: "what value should these caps be?"
- note removed: "10kΩ"
- note removed: "53.6kΩ"
- note removed: "r1"
- note removed: "r2"
- moved on the sheet: C2, C22, C23, C24, C25, C26, C29, C30, C31, C32, C33, C5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

Commit message: ready for review the twost
Other:
- note removed: "what value should these caps be?"
Changed lines of the file:
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@@
 	(generator_version "9.0")
 	(paper "A4")
-	(text "what value should these caps be? "
-		(exclude_from_sim no)
-		(at 172.974 51.308 0)
-		(effects
-			(font
-				(size 1.27 1.27)
-			)
-		)
-	)
 	(text "R2 = 10.0kΩ + R1 = 53.6kΩ"
 		(exclude_from_sim no)

Commit message: ready
Parts:
- C22, C23, C24, C26, C29, C30: footprint Capacitor_SMD:C_0402_1005Metric -> Capacitor_SMD:C_0603_1608Metric
Changed lines of the file:
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@@
 			)
 		)
-		(property "Footprint" "Capacitor_SMD:C_0402_1005Metric"
+		(property "Footprint" "Capacitor_SMD:C_0603_1608Metric"
 			(at 58.7248 83.82 0)
 			(effects
@@
 			)
 		)
-		(property "Footprint" "Capacitor_SMD:C_0402_1005Metric"
+		(property "Footprint" "Capacitor_SMD:C_0603_1608Metric"
 			(at 121.6152 68.58 0)
 			(effects
@@
 			)
 		)
-		(property "Footprint" "Capacitor_SMD:C_0402_1005Metric"
+		(property "Footprint" "Capacitor_SMD:C_0603_1608Metric"
 			(at 134.3152 68.58 0)
 			(effects
@@
 			)
 		)
-		(property "Footprint" "Capacitor_SMD:C_0402_1005Metric"
+		(property "Footprint" "Capacitor_SMD:C_0603_1608Metric"
 			(at 140.6652 68.58 0)
 			(effects
@@
 			)
 		)
-		(property "Footprint" "Capacitor_SMD:C_0402_1005Metric"
+		(property "Footprint" "Capacitor_SMD:C_0603_1608Metric"
 			(at 65.0748 83.82 0)
 			(effects
@@
 			)
 		)
-		(property "Footprint" "Capacitor_SMD:C_0402_1005Metric"
+		(property "Footprint" "Capacitor_SMD:C_0603_1608Metric"
 			(at 127.9652 68.58 0)
 			(effects
